File: flight_computer/flight_computer.kicad_sch (KiCad schematic)
At the start: 0 parts

Commit message: Schematic connecting
Connections:
- no-connect marks 0 -> 4
Other:
- sheet IMU ports: added {I2C}; removed SCL, SDA
- sheet Microcontroller ports: added IMU_FSYNC, RADIO_M0, RADIO_M1, {I2C}; removed IMU_FSYNCH, SCL, SDA
- sheet Pressure sensor ports: added {I2C}; removed SCL, SDA

Commit message: Part way through review
Other:
- sheet Pressure sensor ports: added 1V8A; removed 3V3A
Changed lines of the file:
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@@
   (junction (at 132.08 107.95) (diameter 0) (color 0 0 0 0)
-  )
-  (junction (at 138.43 110.49) (diameter 0) (color 0 0 0 0)
   )
   (no_connect (at 99.06 120.65))
@@
     (stroke (width 0) (type default))
   )
-  (wire (pts (xy 138.43 110.49) (xy 147.32 110.49))
+  (wire (pts (xy 90.17 110.49) (xy 147.32 110.49))
     (stroke (width 0) (type default))
   )
@@
     (stroke (width 0) (type default))
   )
+  (wire (pts (xy 226.06 105.41) (xy 236.22 105.41))
+    (stroke (width 0) (type default))
+  )
   (wire (pts (xy 90.17 105.41) (xy 111.76 105.41))
     (stroke (width 0) (type default))
@@
     (stroke (width 0) (type default))
   )
-  (wire (pts (xy 90.17 110.49) (xy 138.43 110.49))
-    (stroke (width 0) (type default))
-  )
   (wire (pts (xy 132.08 95.25) (xy 226.06 95.25))
     (stroke (width 0) (type default))
@@
     (stroke (width 0) (type default))
   )
-  (wire (pts (xy 138.43 110.49) (xy 138.43 97.79))
-    (stroke (width 0) (type default))
-  )
   (wire (pts (xy 184.15 109.22) (xy 201.93 109.22))
     (stroke (width 0) (type default))
@@
     (stroke (width 0) (type default))
   )
-  (wire (pts (xy 222.25 97.79) (xy 222.25 105.41))
-    (stroke (width 0) (type default))
-  )
   (wire (pts (xy 96.52 182.88) (xy 138.43 182.88))
     (stroke (width 0) (type default))
@@
     (stroke (width 0) (type default))
   )
-  (wire (pts (xy 222.25 105.41) (xy 236.22 105.41))
-    (stroke (width 0) (type default))
-  )
   (wire (pts (xy 90.17 115.57) (xy 147.32 115.57))
     (stroke (width 0) (type default))
@@
     (stroke (width 0) (type default))
   )
-  (wire (pts (xy 138.43 97.79) (xy 222.25 97.79))
-    (stroke (width 0) (type default))
-  )
   (wire (pts (xy 147.32 170.18) (xy 138.43 170.18))
     (stroke (width 0) (type default))
@@
     (effects (font (size 1.27 1.27)) (justify right bottom))
   )
+  (label "1V8A" (at 226.06 105.41 0) (fields_autoplaced)
+    (effects (font (size 1.27 1.27)) (justify left bottom))
+  )
   (label "1V8A" (at 111.76 105.41 180) (fields_autoplaced)
     (effects (font (size 1.27 1.27)) (justify right bottom))
@@
   (label "RADIO_M1" (at 201.93 149.86 180) (fields_autoplaced)
     (effects (font (size 1.27 1.27)) (justify right bottom))
-  )
-  (label "3V3D" (at 106.68 107.95 0) (fields_autoplaced)
-    (effects (font (size 1.27 1.27)) (justify left bottom))
   )
   (symbol (lib_id "power:GND") (at 177.8 182.88 0) (unit 1)
@@
         )
         (path "/89a81c02-14e9-456f-a334-ff69a24bd093"
-          (reference "#PWR011") (unit 1)
+          (reference "#PWR01") (unit 1)
         )
       )
@@
       (effects (font (size 1.27 1.27)) (justify left top))
     )
-    (pin "3V3A" input (at 236.22 105.41 180)
-      (effects (font (size 1.27 1.27)) (justify left))
-    )
     (pin "GND" input (at 236.22 129.54 180)
       (effects (font (size 1.27 1.27)) (justify left))
@@
       (effects (font (size 1.27 1.27)) (justify left))
     )
+    (pin "1V8A" input (at 236.22 105.41 180)
+      (effects (font (size 1.27 1.27)) (justify left))
+    )

Commit message: Thermocouple circuit done
Parts:
- added J5: 3817564, my_footprints:3817564, symbol my_library:3817564
Connections:
- net GND: now also J5.MH1
- new net Temperature sensor/T+: J5.1
- new net Temperature sensor/T-: J5.2
Other:
- sheet Microcontroller ports: added SPI_MISO, SPI_SCK, TC_CS; removed none
- sheet Temperature sensor ports: added 3V3D, GND, SPI_MISO, SPI_SCK, T+, T-, TC_CS; removed none
