File: flight_computer/flight_computer.kicad_sch (KiCad schematic)
At the start: 1 part, among them J5 3817564

Commit message: Layout first effort done
Parts:
- added H1, H2, H3, H4: MountingHole_Pad, MountingHole:MountingHole_3.2mm_M3_Pad_Via, symbol Mechanical:MountingHole_Pad
Connections:
- net GND: now also H1.1, H2.1, H3.1, H4.1
Changed lines of the file:
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@@
   (junction (at 308.61 180.34) (diameter 0) (color 0 0 0 0)
   )
+  (junction (at 313.69 180.34) (diameter 0) (color 0 0 0 0)
+  )
   (junction (at 265.43 180.34) (diameter 0) (color 0 0 0 0)
   )
+  (junction (at 196.85 180.34) (diameter 0) (color 0 0 0 0)
+  )
+  (junction (at 234.95 180.34) (diameter 0) (color 0 0 0 0)
+  )
   (junction (at 228.6 180.34) (diameter 0) (color 0 0 0 0)
   )
@@
   )
   (junction (at 342.9 180.34) (diameter 0) (color 0 0 0 0)
+  )
+  (junction (at 271.78 180.34) (diameter 0) (color 0 0 0 0)
   )
   (junction (at 307.34 92.71) (diameter 0) (color 0 0 0 0)
@@
     (stroke (width 0) (type default))
   )
-  (wire (pts (xy 187.96 180.34) (xy 228.6 180.34))
+  (wire (pts (xy 187.96 180.34) (xy 196.85 180.34))
     (stroke (width 0) (type default))
   )
@@
     (stroke (width 0) (type default))
   )
-  (wire (pts (xy 265.43 180.34) (xy 308.61 180.34))
+  (wire (pts (xy 265.43 180.34) (xy 271.78 180.34))
     (stroke (width 0) (type default))
   )
@@
     (stroke (width 0) (type default))
   )
+  (wire (pts (xy 234.95 180.34) (xy 265.43 180.34))
+    (stroke (width 0) (type default))
+  )
+  (wire (pts (xy 196.85 180.34) (xy 228.6 180.34))
+    (stroke (width 0) (type default))
+  )
+  (wire (pts (xy 271.78 180.34) (xy 308.61 180.34))
+    (stroke (width 0) (type default))
+  )
   (wire (pts (xy 365.76 109.22) (xy 379.73 109.22))
     (stroke (width 0) (type default))
@@
     (stroke (width 0) (type default))
   )
-  (wire (pts (xy 342.9 180.34) (xy 308.61 180.34))
+  (wire (pts (xy 342.9 180.34) (xy 313.69 180.34))
     (stroke (width 0) (type default))
   )
@@
     (stroke (width 0) (type default))
   )
-  (wire (pts (xy 228.6 180.34) (xy 265.43 180.34))
+  (wire (pts (xy 228.6 180.34) (xy 234.95 180.34))
     (stroke (width 0) (type default))
   )
@@
     (stroke (width 0) (type default))
   )
+  (wire (pts (xy 313.69 180.34) (xy 308.61 180.34))
+    (stroke (width 0) (type default))
+  )
   (wire (pts (xy 45.72 113.03) (xy 102.87 113.03))
     (stroke (width 0) (type default))
@@
     (effects (font (size 1.27 1.27)) (justify left bottom))
   )
+  (symbol (lib_id "Mechanical:MountingHole_Pad") (at 196.85 182.88 180) (unit 1)
+    (in_bom no) (on_board yes) (dnp no) (fields_autoplaced)
+    (property "Reference" "H1" (at 199.39 182.88 0)
+      (effects (font (size 1.27 1.27)) (justify right))
+    )
+    (property "Value" "MountingHole_Pad" (at 199.39 185.42 0)
+      (effects (font (size 1.27 1.27)) (justify right))
+    )
+    (property "Footprint" "MountingHole:MountingHole_3.2mm_M3_Pad_Via" (at 196.85 182.88 0)
+      (effects (font (size 1.27 1.27)) hide)
+    )
+    (property "Datasheet" "~" (at 196.85 182.88 0)
+      (effects (font (size 1.27 1.27)) hide)
+    )
+    (property "Manufacturer PN" "~" (at 196.85 182.88 0)
+      (effects (font (size 1.27 1.27)) hide)
+    )
+    (property "Supplier PN" "~" (at 196.85 182.88 0)
+      (effects (font (size 1.27 1.27)) hide)
+    )
+    (property "Supplier" "~" (at 196.85 182.88 0)
+      (effects (font (size 1.27 1.27)) hide)
+    )
+    (pin "1")
+    (instances
+      (project "flight_computer"
+        (path "/89a81c02-14e9-456f-a334-ff69a24bd093"
+          (reference "H1") (unit 1)
+        )
+      )
+    )
+  )
+  (symbol (lib_id "Mechanical:MountingHole_Pad") (at 271.78 182.88 180) (unit 1)
+    (in_bom no) (on_board yes) (dnp no) (fields_autoplaced)
+    (property "Reference" "H3" (at 274.32 182.88 0)
+      (effects (font (size 1.27 1.27)) (justify right))
+    )
+    (property "Value" "MountingHole_Pad" (at 274.32 185.42 0)
+      (effects (font (size 1.27 1.27)) (justify right))
+    )
+    (property "Footprint" "MountingHole:MountingHole_3.2mm_M3_Pad_Via" (at 271.78 182.88 0)
+      (effects (font (size 1.27 1.27)) hide)
+    )
+    (property "Datasheet" "~" (at 271.78 182.88 0)
+      (effects (font (size 1.27 1.27)) hide)
+    )
+    (property "Manufacturer PN" "~" (at 271.78 182.88 0)
+      (effects (font (size 1.27 1.27)) hide)
+    )
+    (property "Supplier PN" "~" (at 271.78 182.88 0)
+      (effects (font (size 1.27 1.27)) hide)
+    )
+    (property "Supplier" "~" (at 271.78 182.88 0)
+      (effects (font (size 1.27 1.27)) hide)
+    )
+    (pin "1")
+    (instances
+      (project "flight_computer"
+        (path "/89a81c02-14e9-456f-a334-ff69a24bd093"
+          (reference "H3") (unit 1)
+        )
+      )
+    )
+  )
+  (symbol (lib_id "Mechanical:MountingHole_Pad") (at 234.95 182.88 180) (unit 1)
+    (in_bom no) (on_board yes) (dnp no) (fields_autoplaced)
+    (property "Reference" "H2" (at 237.49 182.88 0)
+      (effects (font (size 1.27 1.27)) (justify right))
+    )
+    (property "Value" "MountingHole_Pad" (at 237.49 185.42 0)
+      (effects (font (size 1.27 1.27)) (justify right))
+    )
+    (property "Footprint" "MountingHole:MountingHole_3.2mm_M3_Pad_Via" (at 234.95 182.88 0)
+      (effects (font (size 1.27 1.27)) hide)
+    )
+    (property "Datasheet" "~" (at 234.95 182.88 0)
+      (effects (font (size 1.27 1.27)) hide)
+    )
+    (property "Manufacturer PN" "~" (at 234.95 182.88 0)
+      (effects (font (size 1.27 1.27)) hide)
+    )
+    (property "Supplier PN" "~" (at 234.95 182.88 0)
+      (effects (font (size 1.27 1.27)) hide)
+    )
+    (property "Supplier" "~" (at 234.95 182.88 0)
+      (effects (font (size 1.27 1.27)) hide)
+    )
+    (pin "1")
+    (instances
+      (project "flight_computer"
+        (path "/89a81c02-14e9-456f-a334-ff69a24bd093"
+          (reference "H2") (unit 1)
+        )
+      )
+    )
+  )
+  (symbol (lib_id "Mechanical:MountingHole_Pad") (at 313.69 182.88 180) (unit 1)
+    (in_bom no) (on_board yes) (dnp no) (fields_autoplaced)
+    (property "Reference" "H4" (at 316.23 182.88 0)
+      (effects (font (size 1.27 1.27)) (justify right))
+    )
+    (property "Value" "MountingHole_Pad" (at 316.23 185.42 0)
+      (effects (font (size 1.27 1.27)) (justify right))
+    )
+    (property "Footprint" "MountingHole:MountingHole_3.2mm_M3_Pad_Via" (at 313.69 182.88 0)
+      (effects (font (size 1.27 1.27)) hide)
+    )
+    (property "Datasheet" "~" (at 313.69 182.88 0)
+      (effects (font (size 1.27 1.27)) hide)
+    )
+    (property "Manufacturer PN" "~" (at 313.69 182.88 0)
+      (effects (font (size 1.27 1.27)) hide)
+    )
+    (property "Supplier PN" "~" (at 313.69 182.88 0)
+      (effects (font (size 1.27 1.27)) hide)
+    )
+    (property "Supplier" "~" (at 313.69 182.88 0)
+      (effects (font (size 1.27 1.27)) hide)
+    )
+    (pin "1")
+    (instances
+      (project "flight_computer"
+        (path "/89a81c02-14e9-456f-a334-ff69a24bd093"
+          (reference "H4") (unit 1)
+        )
+      )
+    )
+  )
   (symbol (lib_id "power:GND") (at 133.35 180.34 0) (unit 1)

Commit message: Adding SDCC user manual annotated and some makefile notes
Parts:
- J5: Manufacturer PN (none) -> 3817564; Supplier (none) -> RS; Supplier PN (none) -> 3817564; now left out of the parts list
Changed lines of the file:
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@@
   )
   (symbol (lib_id "my_library:3817564") (at 354.33 107.95 0) (unit 1)
-    (in_bom yes) (on_board yes) (dnp no) (fields_autoplaced)
+    (in_bom no) (on_board yes) (dnp no) (fields_autoplaced)
     (property "Reference" "J5" (at 354.33 99.06 0)
       (effects (font (size 1.27 1.27)))
@@
       (effects (font (size 1.27 1.27)) (justify left top) hide)
     )
+    (property "Manufacturer PN" "3817564" (at 354.33 107.95 0)
+      (effects (font (size 1.27 1.27)) hide)
+    )
+    (property "Supplier PN" "3817564" (at 354.33 107.95 0)
+      (effects (font (size 1.27 1.27)) hide)
+    )
+    (property "Supplier" "RS" (at 354.33 107.95 0)
+      (effects (font (size 1.27 1.27)) hide)
+    )
     (pin "1")

Commit message: RevB PCB work
Other:
- sheet Microcontroller ports: added VBUS_5V_IN; removed none
Changed lines of the file:
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@@
+    (stroke (width 0) (type default))
+  )
+  (wire (pts (xy 88.9 121.92) (xy 102.87 121.92))
     (stroke (width 0) (type default))
   )
@@
       (effects (font (size 1.27 1.27)) (justify right))
     )
-    (instances
+    (pin "VBUS_5V_IN" output (at 102.87 121.92 180)
+      (effects (font (size 1.27 1.27)) (justify left))
+    )
+    (instances
