File: flight_computer/temp_sensor.kicad_sch (KiCad schematic)
At the start: 0 parts

Commit message: Adding shauns thermcoouple
Parts:
- added C1 (x3): 100nF, Capacitor_SMD:C_0402_1005Metric, symbol Device:C
- added C24: 1uF, Capacitor_SMD:C_0402_1005Metric, symbol Device:C
- added R21, R23: 150R, Resistor_SMD:R_0402_1005Metric, symbol Device:R
- added U8: MAX31855KASA, Package_SO:SOIC-8_3.9x4.9mm_P1.27mm, symbol Sensor_Temperature:MAX31855KASA
Connections:
- new net: C1.1, C24.2, R23.2, U8.2 (T-)
- new net: C1.2, C24.1, R21.2, U8.3 (T+)
- new net 3V3D: C1.1, U8.4 (V_CC)
- new net GND: C1.1, C1.2, C1.2, U8.1 (GND)
- new net SPI_MISO: U8.7 (SO)
- new net SPI_NSS: U8.6 (~{CS})
- new net SPI_SCK: U8.5 (SCK)
- new net T+: R21.1
- new net T-: R23.1
Other:
- note added: "1 kHz common mode LPF"
- note added: "32 MHz differential mode LPF"
- note added: "Thermocouple"

Commit message: Thermocouple circuit done
Connections:
- net SPI_NSS renamed TC_CS
Changed lines of the file:
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@@
-    (effects (font (size 1.27 1.27)) (justify left bottom))
-  )
-  (label "SPI_NSS" (at 185.42 96.52 0) (fields_autoplaced)
-    (effects (font (size 1.27 1.27)) (justify left bottom))
-  )
-  (label "SPI_MISO" (at 185.42 91.44 0) (fields_autoplaced)
-    (effects (font (size 1.27 1.27)) (justify left bottom))
-  )
-  (label "SPI_SCK" (at 185.42 88.9 0) (fields_autoplaced)
     (effects (font (size 1.27 1.27)) (justify left bottom))
   )
@@
     (effects (font (size 1.27 1.27)) (justify right))
   )
+  (hierarchical_label "TC_CS" (shape input) (at 185.42 96.52 0) (fields_autoplaced)
+    (effects (font (size 1.27 1.27)) (justify left))
+  )
+  (hierarchical_label "SPI_MISO" (shape output) (at 185.42 91.44 0) (fields_autoplaced)
+    (effects (font (size 1.27 1.27)) (justify left))
+  )
   (hierarchical_label "GND" (shape input) (at 93.98 120.65 180) (fields_autoplaced)
     (effects (font (size 1.27 1.27)) (justify right))
   )
+  (hierarchical_label "SPI_SCK" (shape input) (at 185.42 88.9 0) (fields_autoplaced)
+    (effects (font (size 1.27 1.27)) (justify left))
+  )
   (symbol (lib_id "Device:C") (at 99.06 95.25 0) (unit 1)
