File: flight_computer/flight_computer.kicad_pcb (KiCad board)
At the start: 2 copper layers, 89 parts, among them J1 Conn_02x05_Odd_Even, J2 MEM2061-01-188-00-A_REVA, J3 Conn_01x02, J4 Conn_01x07, J5 3817564, Q1 Q_NPN_BEC, Q2 Q_NMOS_GSD, SW1 SW_Push, SW2 SW_Push, U1 STM8S007C8T6TR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

Commit message: testing kicad version compatibility
Parts:
- moved C33 34.6 mm to (153.0, 138.5)
- moved C34 30.2 mm to (164.0, 138.5)
- moved U8 29.6 mm to (179.0, 137.4)
- moved R25 29.2 mm to (159.5, 142.5)
- moved C36 28.5 mm to (168.3, 140.8)
- moved C35 24.7 mm to (168.5, 135.0)
- moved R24 24.5 mm to (159.5, 135.5)

Commit message: KiCAD8 is not compatible with 7: Revert "testing kicad version compatibility"
This reverts commit 37378f71d3b59c33c1abc1999dff2b71273f3631.
Parts:
- moved C33 34.6 mm to (166.2, 106.5)
- moved C34 30.2 mm to (166.2, 108.4)
- moved U8 29.6 mm to (171.8, 108.7)
- moved R25 29.2 mm to (169.1, 114.9)
- moved C36 28.5 mm to (166.2, 112.4)
- moved C35 24.7 mm to (166.2, 110.4)
- moved R24 24.5 mm to (169.1, 112.9)

Commit message: A hearty attempt at CPU wiring.
Parts:
- moved C4 93.3 mm to (101.6, 137.1)
- moved C2 92.8 mm to (98.0, 131.9), turned to 180 degrees
- moved C3 89.3 mm to (101.7, 138.0)
- moved C1 88.1 mm to (97.2, 130.9), turned to 180 degrees
- moved C10 88.0 mm to (96.4, 133.4), turned to -90 degrees
- moved C11 87.3 mm to (95.5, 133.4), turned to -90 degrees
- moved C8 86.0 mm to (98.5, 133.4), turned to -90 degrees
- moved C9 85.2 mm to (97.4, 133.4), turned to -90 degrees
- moved C7 85.2 mm to (98.5, 130.4), turned to 90 degrees
- moved U1 66.4 mm to (104.2, 131.3)
Routing:
- net GND: track 0.00 -> 14.5 mm
- net /Microcontroller/3V3D: track 0.00 -> 8.09 mm
- net /Power/3V3A: track 0.00 -> 2.71 mm
- net Net-(U1B-VCAP): track 0.00 -> 1.73 mm

Commit message: Start of layout
Parts:
- C1, C10, C11, C17, C19, C20, C22, C3: footprint Capacitor_SMD:C_0201_0603Metric -> Capacitor_SMD:C_0402_1005Metric
- C7: moved to B.Cu
- moved J2 129.2 mm to (246.3, 141.9)
- moved R8 114.8 mm to (255.0, 122.0)
- moved R7 114.7 mm to (255.0, 119.7)
- moved J5 99.2 mm to (266.1, 58.7)
- moved Q1 97.2 mm to (251.1, 121.2)
- moved R3 96.6 mm to (240.0, 100.8)
- moved BZ1 96.1 mm to (244.3, 121.0)
- moved SW1 91.3 mm to (241.7, 98.8)
- moved R6 89.2 mm to (238.1, 89.7)
- moved C12 87.4 mm to (240.0, 89.7)
- moved SW2 84.2 mm to (240.0, 87.7)
- moved R16 79.4 mm to (192.7, 49.6)
- moved C18 73.2 mm to (188.7, 47.4), turned to 90 degrees
- moved L1 70.2 mm to (187.5, 56.3), turned to 180 degrees
- moved U3 70.1 mm to (187.9, 50.2), turned to 90 degrees
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Routing:
- net GND: track 14.5 -> 44.8 mm, vias 0 -> 20
- net /Microcontroller/3V3D: track 8.09 -> 27.4 mm, vias 0 -> 11
- net /1V8A: track 0.00 -> 6.87 mm, vias 0 -> 4
- net Net-(U1A-PA2/OSCOUT): track 0.00 -> 6.78 mm
- net Net-(U1A-PA1/OSCIN): track 0.00 -> 6.40 mm
- net Net-(U3-L1): track 0.00 -> 3.23 mm, vias 0 -> 2
- net Net-(U3-L2): track 0.00 -> 1.78 mm, vias 0 -> 2
- net /Power/3V3A: track 2.71 -> 4.16 mm, vias 0 -> 2
- net Net-(U1B-VCAP): track 1.73 -> 1.99 mm, vias 0 -> 1
- added copper zone on F.Cu, net /Microcontroller/3V3D
Other:
- copper layers 2 -> 4
