File: flight_computer/imu.kicad_sch (KiCad schematic)
At the start: 4 parts, among them U6 ICM-42670-P

Commit message: Schematic connecting
Changed lines of the file:
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@@
   (junction (at 127 95.25) (diameter 0) (color 0 0 0 0)
+  )
+  (bus_entry (at 246.38 100.33) (size -2.54 2.54)
+    (stroke (width 0) (type default))
+  )
+  (bus_entry (at 246.38 102.87) (size -2.54 2.54)
+    (stroke (width 0) (type default))
   )
   (wire (pts (xy 82.55 125.73) (xy 102.87 125.73))
@@
     (stroke (width 0) (type default))
   )
+  (wire (pts (xy 203.2 102.87) (xy 243.84 102.87))
+    (stroke (width 0) (type default))
+  )
   (wire (pts (xy 203.2 95.25) (xy 217.17 95.25))
+    (stroke (width 0) (type default))
+  )
+  (bus (pts (xy 255.27 97.79) (xy 246.38 97.79))
     (stroke (width 0) (type default))
   )
@@
     (stroke (width 0) (type default))
   )
-  (wire (pts (xy 203.2 102.87) (xy 217.17 102.87))
+  (wire (pts (xy 203.2 105.41) (xy 243.84 105.41))
     (stroke (width 0) (type default))
   )
   (wire (pts (xy 181.61 125.73) (xy 214.63 125.73))
+    (stroke (width 0) (type default))
+  )
+  (bus (pts (xy 246.38 100.33) (xy 246.38 102.87))
     (stroke (width 0) (type default))
   )
@@
     (stroke (width 0) (type default))
   )
-  (wire (pts (xy 203.2 105.41) (xy 217.17 105.41))
-    (stroke (width 0) (type default))
-  )
   (wire (pts (xy 181.61 121.92) (xy 181.61 125.73))
     (stroke (width 0) (type default))
@@
     (stroke (width 0) (type default))
   )
-  (text "I2C addr LSB=0" (at 215.9 109.22 0)
+  (bus (pts (xy 246.38 97.79) (xy 246.38 100.33))
+    (stroke (width 0) (type default))
+  )
+  (text "I2C addr LSB=0" (at 199.39 110.49 0)
     (effects (font (size 1.27 1.27)) (justify left bottom))
   )
-  (text "Pull to VDDIO for I2C" (at 220.98 100.33 0)
+  (text "Pull to VDDIO for I2C" (at 218.44 100.33 0)
     (effects (font (size 1.27 1.27)) (justify left bottom))
   )
@@
     (effects (font (size 1.27 1.27)) (justify right bottom))
   )
+  (label "SCL" (at 240.03 102.87 180) (fields_autoplaced)
+    (effects (font (size 1.27 1.27)) (justify right bottom))
+  )
+  (label "SDA" (at 240.03 105.41 180) (fields_autoplaced)
+    (effects (font (size 1.27 1.27)) (justify right bottom))
+  )
   (hierarchical_label "3V3D" (shape input) (at 121.92 95.25 180) (fields_autoplaced)
     (effects (font (size 1.27 1.27)) (justify right))
@@
   (hierarchical_label "INT1" (shape output) (at 148.59 100.33 180) (fields_autoplaced)
     (effects (font (size 1.27 1.27)) (justify right))
-  )
-  (hierarchical_label "SDA" (shape bidirectional) (at 217.17 105.41 0) (fields_autoplaced)
-    (effects (font (size 1.27 1.27)) (justify left))
   )
   (hierarchical_label "1V8A" (shape input) (at 71.12 92.71 180) (fields_autoplaced)
@@
     (effects (font (size 1.27 1.27)) (justify left))
   )
-  (hierarchical_label "SCL" (shape input) (at 217.17 102.87 0) (fields_autoplaced)
-    (effects (font (size 1.27 1.27)) (justify left))
-  )
   (hierarchical_label "GND" (shape input) (at 69.85 125.73 180) (fields_autoplaced)
     (effects (font (size 1.27 1.27)) (justify right))
   )
+  (hierarchical_label "{I2C}" (shape input) (at 255.27 97.79 0) (fields_autoplaced)
+    (effects (font (size 1.27 1.27) (thickness 0.254) bold) (justify left))
+  )
   (hierarchical_label "INT2" (shape output) (at 148.59 102.87 180) (fields_autoplaced)

Commit message: ERC complete
Changed lines of the file:
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@@
   (junction (at 127 95.25) (diameter 0) (color 0 0 0 0)
   )
+  (junction (at 162.56 125.73) (diameter 0) (color 0 0 0 0)
+  )
   (bus_entry (at 246.38 100.33) (size -2.54 2.54)
     (stroke (width 0) (type default))
@@
     (stroke (width 0) (type default))
   )
+  (wire (pts (xy 227.33 78.74) (xy 227.33 100.33))
+    (stroke (width 0) (type default))
+  )
   (wire (pts (xy 102.87 92.71) (xy 102.87 104.14))
     (stroke (width 0) (type default))
@@
     (stroke (width 0) (type default))
   )
-  (wire (pts (xy 152.4 125.73) (xy 173.99 125.73))
+  (wire (pts (xy 152.4 125.73) (xy 162.56 125.73))
     (stroke (width 0) (type default))
   )
@@
     (stroke (width 0) (type default))
   )
-  (wire (pts (xy 203.2 100.33) (xy 217.17 100.33))
+  (wire (pts (xy 203.2 100.33) (xy 227.33 100.33))
     (stroke (width 0) (type default))
   )
@@
     (stroke (width 0) (type default))
   )
+  (wire (pts (xy 162.56 125.73) (xy 173.99 125.73))
+    (stroke (width 0) (type default))
+  )
   (wire (pts (xy 102.87 111.76) (xy 102.87 125.73))
+    (stroke (width 0) (type default))
+  )
+  (wire (pts (xy 127 95.25) (xy 127 78.74))
+    (stroke (width 0) (type default))
+  )
+  (wire (pts (xy 127 78.74) (xy 227.33 78.74))
     (stroke (width 0) (type default))
   )
@@
   (text "Pull to VDDIO for I2C" (at 218.44 100.33 0)
     (effects (font (size 1.27 1.27)) (justify left bottom))
-  )
-  (label "VDDIO" (at 129.54 95.25 0) (fields_autoplaced)
-    (effects (font (size 1.27 1.27)) (justify left bottom))
-  )
-  (label "VDDIO" (at 217.17 100.33 180) (fields_autoplaced)
-    (effects (font (size 1.27 1.27)) (justify right bottom))
   )
   (label "SCL" (at 240.03 102.87 180) (fields_autoplaced)
@@
         )
       )
+    )
+  )
+  (symbol (lib_id "power:GND") (at 162.56 125.73 0) (unit 1)
+    (in_bom yes) (on_board yes) (dnp no) (fields_autoplaced)
+    (property "Reference" "#PWR015" (at 162.56 132.08 0)
+      (effects (font (size 1.27 1.27)) hide)
+    )
+    (property "Value" "GND" (at 162.56 130.81 0)
+      (effects (font (size 1.27 1.27)))
+    )
+    (property "Footprint" "" (at 162.56 125.73 0)
+      (effects (font (size 1.27 1.27)) hide)
+    )
+    (property "Datasheet" "" (at 162.56 125.73 0)
+      (effects (font (size 1.27 1.27)) hide)
+    )
+    (pin "1")
+    (instances
+      (project "flight_computer"
+        (path "/89a81c02-14e9-456f-a334-ff69a24bd093/ebc948db-a9d3-410a-bdbf-1c31db890e56"
+          (reference "#PWR015") (unit 1)
+        )
+        (path "/89a81c02-14e9-456f-a334-ff69a24bd093"
+          (reference "#PWR011") (unit 1)
+        )
+        (path "/89a81c02-14e9-456f-a334-ff69a24bd093/00230fc6-00d9-4789-9199-c0e29b2f6daa"
+          (reference "#PWR016") (unit 1)
+        )
+      )

Commit message: Part way through review
Parts:
- U7: renamed from U6; Supplier (none) -> Digikey; Supplier PN (none) -> 1428-ICM-42670-PCT-ND
- renumbered C19 to C23, C18 to C24
Changed lines of the file:
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@@
   (symbol (lib_id "Device:C") (at 102.87 107.95 0) (unit 1)
     (in_bom yes) (on_board yes) (dnp no)
-    (property "Reference" "C19" (at 106.68 106.68 0)
+    (property "Reference" "C23" (at 106.68 106.68 0)
       (effects (font (size 1.27 1.27)) (justify left))
     )
@@
       (project "flight_computer"
         (path "/89a81c02-14e9-456f-a334-ff69a24bd093/00230fc6-00d9-4789-9199-c0e29b2f6daa"
-          (reference "C19") (unit 1)
+          (reference "C23") (unit 1)
         )
       )
@@
   (symbol (lib_id "Device:C") (at 127 107.95 0) (unit 1)
     (in_bom yes) (on_board yes) (dnp no)
-    (property "Reference" "C18" (at 130.81 106.68 0)
+    (property "Reference" "C24" (at 130.81 106.68 0)
       (effects (font (size 1.27 1.27)) (justify left))
     )
@@
       (project "flight_computer"
         (path "/89a81c02-14e9-456f-a334-ff69a24bd093/00230fc6-00d9-4789-9199-c0e29b2f6daa"
-          (reference "C18") (unit 1)
+          (reference "C24") (unit 1)
         )
       )
@@
   (symbol (lib_id "my_library:ICM-42670-P") (at 177.8 100.33 0) (unit 1)
     (in_bom yes) (on_board yes) (dnp no) (fields_autoplaced)
-    (property "Reference" "U6" (at 177.8 82.55 0)
+    (property "Reference" "U7" (at 177.8 82.55 0)
       (effects (font (size 1.27 1.27)))
     )
@@
     )
     (property "Manufacturer PN" "ICM-42670-P" (at 179.07 81.28 0)
+      (effects (font (size 1.27 1.27)) hide)
+    )
+    (property "Supplier" "Digikey" (at 177.8 100.33 0)
+      (effects (font (size 1.27 1.27)) hide)
+    )
+    (property "Supplier PN" "1428-ICM-42670-PCT-ND" (at 177.8 100.33 0)
       (effects (font (size 1.27 1.27)) hide)
     )
@@
       (project "flight_computer"
         (path "/89a81c02-14e9-456f-a334-ff69a24bd093/00230fc6-00d9-4789-9199-c0e29b2f6daa"
-          (reference "U6") (unit 1)
+          (reference "U7") (unit 1)
         )
       )
@@
         )
         (path "/89a81c02-14e9-456f-a334-ff69a24bd093/00230fc6-00d9-4789-9199-c0e29b2f6daa"
-          (reference "C17") (unit 1)
+          (reference "C22") (unit 1)
         )
       )

Commit message: Adding shauns thermcoouple
Parts:
- renumbered C23 to C31, C24 to C32
Changed lines of the file:
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@@
   (symbol (lib_id "Device:C") (at 102.87 107.95 0) (unit 1)
     (in_bom yes) (on_board yes) (dnp no)
-    (property "Reference" "C23" (at 106.68 106.68 0)
+    (property "Reference" "C31" (at 106.68 106.68 0)
       (effects (font (size 1.27 1.27)) (justify left))
     )
@@
       (project "flight_computer"
         (path "/89a81c02-14e9-456f-a334-ff69a24bd093/00230fc6-00d9-4789-9199-c0e29b2f6daa"
-          (reference "C23") (unit 1)
+          (reference "C31") (unit 1)
         )
       )
@@
   (symbol (lib_id "Device:C") (at 127 107.95 0) (unit 1)
     (in_bom yes) (on_board yes) (dnp no)
-    (property "Reference" "C24" (at 130.81 106.68 0)
+    (property "Reference" "C32" (at 130.81 106.68 0)
       (effects (font (size 1.27 1.27)) (justify left))
     )
@@
       (project "flight_computer"
         (path "/89a81c02-14e9-456f-a334-ff69a24bd093/00230fc6-00d9-4789-9199-c0e29b2f6daa"
-          (reference "C24") (unit 1)
+          (reference "C32") (unit 1)
         )
       )
@@
         )
         (path "/89a81c02-14e9-456f-a334-ff69a24bd093/00230fc6-00d9-4789-9199-c0e29b2f6daa"
-          (reference "C22") (unit 1)
+          (reference "C30") (unit 1)
         )
       )
