File: flight_computer/gps.kicad_sch (KiCad schematic)
At the start: 9 parts, among them U6 YIC31612EBGG, U9 Antenna_GPS

Commit message: ERC okay
Connections:
- net GND: now also U9.5 (CAP)
Changed lines of the file:
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@@
   (junction (at 85.09 87.63) (diameter 0) (color 0 0 0 0)
+  )
+  (junction (at 105.41 119.38) (diameter 0) (color 0 0 0 0)
   )
   (junction (at 68.58 119.38) (diameter 0) (color 0 0 0 0)
@@
     (stroke (width 0) (type default))
   )
+  (wire (pts (xy 105.41 119.38) (xy 146.05 119.38))
+    (stroke (width 0) (type default))
+  )
   (wire (pts (xy 151.13 119.38) (xy 153.67 119.38))
     (stroke (width 0) (type default))
@@
     (stroke (width 0) (type default))
   )
-  (wire (pts (xy 102.87 119.38) (xy 146.05 119.38))
+  (wire (pts (xy 102.87 119.38) (xy 105.41 119.38))
     (stroke (width 0) (type default))
   )
@@
   )
   (wire (pts (xy 130.81 96.52) (xy 135.89 96.52))
+    (stroke (width 0) (type default))
+  )
+  (wire (pts (xy 105.41 113.03) (xy 105.41 119.38))
     (stroke (width 0) (type default))
   )
@@
     (pin "3")
     (pin "4")
-    (instances
-      (project "flight_computer"
+    (pin "5")
+    (instances
+      (project "flight_computer"

Commit message: Adding SDCC user manual annotated and some makefile notes
Parts:
- U9: Manufacturer PN (none) -> 1582AT54A0045; Supplier (none) -> Digikey; Supplier PN (none) -> 712-1582AT54A0045001ECT-ND
Changed lines of the file:
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@@
       (effects (font (size 1.27 1.27)) hide)
     )
-    (property "Manufacturer PN" "" (at 102.87 104.14 0)
+    (property "Manufacturer PN" "1582AT54A0045" (at 102.87 104.14 0)
       (effects (font (size 1.27 1.27)) hide)
     )
-    (property "Supplier PN" "" (at 102.87 104.14 0)
+    (property "Supplier PN" "712-1582AT54A0045001ECT-ND" (at 102.87 104.14 0)
       (effects (font (size 1.27 1.27)) hide)
     )
-    (property "Supplier" "" (at 102.87 104.14 0)
+    (property "Supplier" "Digikey" (at 102.87 104.14 0)
       (effects (font (size 1.27 1.27)) hide)
     )
